Commit message: Changes on urdf and added a robot launch file.

File: robots/g1_description/g1_29dof_lock_waist_with_hand_rev_1_0.urdf (robot description, URDF)
Before this commit: robot g1_29dof_lock_waist_with_hand_rev_1_0, 53 links, 52 joints
Links:
- added link base_link
- link head_link: geometry collision mesh filename=/unitree/livox_mapping/robots/g1_description/meshes/head_li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; visual mesh filename=/unitree/livox_mapping/robots/g1_description/meshes/head_li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
- link left_ankle_pitch_link: geometry collision mesh filename=/unitree/livox_mapping/robots/g1_description/meshes/left_an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; visual mesh filename=/unitree/livox_mapping/robots/g1_description/meshes/left_an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
- link left_ankle_roll_link: geometry collision sphere radius=0.005; collision sphere radius=0.005
- link left_elbow_link: geometry collision mesh filename=/unitree/livox_mapping/robots/g1_description/meshes/left_el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; visual mesh filename=/unitree/livox_mapping/robots/g1_description/meshes/left_el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
- link left_hand_index_0_link: geometry collision mesh filename=/unitree/livox_mapping/robots/g1_description/meshes/left_ha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; visual mesh filename=/unitree/livox_mapping/robots/g1_description/meshes/left_ha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
- link left_hand_index_1_link: geometry collision mesh filename=/unitree/livox_mapping/robots/g1_description/meshes/left_ha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; visual mesh filename=/unitree/livox_mapping/robots/g1_description/meshes/left_ha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
- link left_hand_middle_0_link: geometry collision mesh filename=/unitree/livox_mapping/robots/g1_description/meshes/left_ha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; visual mesh filename=/unitree/livox_mapping/robots/g1_description/meshes/left_ha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
- link left_hand_middle_1_link: geometry collision mesh filename=/unitree/livox_mapping/robots/g1_description/meshes/left_ha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; visual mesh filename=/unitree/livox_mapping/robots/g1_description/meshes/left_ha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
- link left_hand_palm_link: geometry collision mesh filename=/unitree/livox_mapping/robots/g1_description/meshes/left_ha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; visual mesh filename=/unitree/livox_mapping/robots/g1_description/meshes/left_ha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
- link left_hand_thumb_0_link: geometry collision mesh filename=/unitree/livox_mapping/robots/g1_description/meshes/left_ha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; visual mesh filename=/unitree/livox_mapping/robots/g1_description/meshes/left_ha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
- link left_hand_thumb_1_link: geometry collision box size=0.02 0.03 0.02; visual mesh filename=/unitree/livox_mapping/robots/g1_description/meshes/left_ha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
- link left_hand_thumb_2_link: geometry collision mesh filename=/unitree/livox_mapping/robots/g1_description/meshes/left_ha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; visual mesh filename=/unitree/livox_mapping/robots/g1_description/meshes/left_ha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
- link left_hip_pitch_link: geometry collision mesh filename=/unitree/livox_mapping/robots/g1_description/meshes/left_hi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; visual mesh filename=/unitree/livox_mapping/robots/g1_description/meshes/left_hi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
- link left_hip_roll_link: geometry collision mesh filename=/unitree/livox_mapping/robots/g1_description/meshes/left_hi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; visual mesh filename=/unitree/livox_mapping/robots/g1_description/meshes/left_hi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
- link left_hip_yaw_link: geometry collision mesh filename=/unitree/livox_mapping/robots/g1_description/meshes/left_hi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; visual mesh filename=/unitree/livox_mapping/robots/g1_description/meshes/left_hi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
- link left_knee_link: geometry collision mesh filename=/unitree/livox_mapping/robots/g1_description/meshes/left_kn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; visual mesh filename=/unitree/livox_mapping/robots/g1_description/meshes/left_kn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
- link left_shoulder_pitch_link: geometry collision cylinder length=0.05 radius=0.03; visual mesh filename=/unitree/livox_mapping/robots/g1_description/meshes/left_sh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
- link left_shoulder_roll_link: geometry collision cylinder length=0.03 radius=0.03; visual mesh filename=/unitree/livox_mapping/robots/g1_description/meshes/left_sh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
- link left_shoulder_yaw_link: geometry collision mesh filename=/unitree/livox_mapping/robots/g1_description/meshes/left_sh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; visual mesh filename=/unitree/livox_mapping/robots/g1_description/meshes/left_sh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
- link left_wrist_pitch_link: geometry collision mesh filename=/unitree/livox_mapping/robots/g1_description/meshes/left_wr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; visual mesh filename=/unitree/livox_mapping/robots/g1_description/meshes/left_wr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
- link left_wrist_roll_link: geometry collision mesh filename=/unitree/livox_mapping/robots/g1_description/meshes/left_wr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; visual mesh filename=/unitree/livox_mapping/robots/g1_description/meshes/left_wr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
- link left_wrist_yaw_link: geometry collision mesh filename=/unitree/livox_mapping/robots/g1_description/meshes/left_wr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; visual mesh filename=/unitree/livox_mapping/robots/g1_description/meshes/left_wr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
- link logo_link: geometry collision mesh filename=/unitree/livox_mapping/robots/g1_description/meshes/logo_li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; visual mesh filename=/unitree/livox_mapping/robots/g1_description/meshes/logo_li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
- link pelvis: geometry visual mesh filename=/unitree/livox_mapping/robots/g1_description/meshes/pelvis.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
- link pelvis_contour_link: geometry collision mesh filename=/unitree/livox_mapping/robots/g1_description/meshes/pelvis_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; visual mesh filename=/unitree/livox_mapping/robots/g1_description/meshes/pelvis_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
- link right_ankle_pitch_link: geometry collision mesh filename=/unitree/livox_mapping/robots/g1_description/meshes/right_a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; visual mesh filename=/unitree/livox_mapping/robots/g1_description/meshes/right_a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
- link right_ankle_roll_link: geometry collision sphere radius=0.005; collision sphere radius=0.005
- link right_elbow_link: geometry collision mesh filename=/unitree/livox_mapping/robots/g1_description/meshes/right_e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; visual mesh filename=/unitree/livox_mapping/robots/g1_description/meshes/right_e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
- link right_hand_index_0_link: geometry collision mesh filename=/unitree/livox_mapping/robots/g1_description/meshes/right_h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; visual mesh filename=/unitree/livox_mapping/robots/g1_description/meshes/right_h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
- link right_hand_index_1_link: geometry collision mesh filename=/unitree/livox_mapping/robots/g1_description/meshes/right_h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; visual mesh filename=/unitree/livox_mapping/robots/g1_description/meshes/right_h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
- link right_hand_middle_0_link: geometry collision mesh filename=/unitree/livox_mapping/robots/g1_description/meshes/right_h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; visual mesh filename=/unitree/livox_mapping/robots/g1_description/meshes/right_h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
- link right_hand_middle_1_link: geometry collision mesh filename=/unitree/livox_mapping/robots/g1_description/meshes/right_h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; visual mesh filename=/unitree/livox_mapping/robots/g1_description/meshes/right_h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
- link right_hand_palm_link: geometry collision mesh filename=/unitree/livox_mapping/robots/g1_description/meshes/right_h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; visual mesh filename=/unitree/livox_mapping/robots/g1_description/meshes/right_h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
- link right_hand_thumb_0_link: geometry collision mesh filename=/unitree/livox_mapping/robots/g1_description/meshes/right_h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; visual mesh filename=/unitree/livox_mapping/robots/g1_description/meshes/right_h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
- link right_hand_thumb_1_link: geometry collision box size=0.02 0.03 0.02; visual mesh filename=/unitree/livox_mapping/robots/g1_description/meshes/right_h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
- link right_hand_thumb_2_link: geometry collision mesh filename=/unitree/livox_mapping/robots/g1_description/meshes/right_h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; visual mesh filename=/unitree/livox_mapping/robots/g1_description/meshes/right_h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
- link right_hip_pitch_link: geometry collision mesh filename=/unitree/livox_mapping/robots/g1_description/meshes/right_h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; visual mesh filename=/unitree/livox_mapping/robots/g1_description/meshes/right_h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
- link right_hip_roll_link: geometry collision mesh filename=/unitree/livox_mapping/robots/g1_description/meshes/right_h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; visual mesh filename=/unitree/livox_mapping/robots/g1_description/meshes/right_h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
- link right_hip_yaw_link: geometry collision mesh filename=/unitree/livox_mapping/robots/g1_description/meshes/right_h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; visual mesh filename=/unitree/livox_mapping/robots/g1_description/meshes/right_h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
- link right_knee_link: geometry collision mesh filename=/unitree/livox_mapping/robots/g1_description/meshes/right_k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; visual mesh filename=/unitree/livox_mapping/robots/g1_description/meshes/right_k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
- link right_shoulder_pitch_link: geometry collision cylinder length=0.05 radius=0.03; visual mesh filename=/unitree/livox_mapping/robots/g1_description/meshes/right_s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
- link right_shoulder_roll_link: geometry collision cylinder length=0.03 radius=0.03; visual mesh filename=/unitree/livox_mapping/robots/g1_description/meshes/right_s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
- link right_shoulder_yaw_link: geometry collision mesh filename=/unitree/livox_mapping/robots/g1_description/meshes/right_s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; visual mesh filename=/unitree/livox_mapping/robots/g1_description/meshes/right_s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
- link right_wrist_pitch_link: geometry collision mesh filename=/unitree/livox_mapping/robots/g1_description/meshes/right_w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; visual mesh filename=/unitree/livox_mapping/robots/g1_description/meshes/right_w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
- link right_wrist_roll_link: geometry collision mesh filename=/unitree/livox_mapping/robots/g1_description/meshes/right_w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; visual mesh filename=/unitree/livox_mapping/robots/g1_description/meshes/right_w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
- link right_wrist_yaw_link: geometry collision mesh filename=/unitree/livox_mapping/robots/g1_description/meshes/right_w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; visual mesh filename=/unitree/livox_mapping/robots/g1_description/meshes/right_w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
- link torso_link: geometry collision mesh filename=/unitree/livox_mapping/robots/g1_description/meshes/torso_l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; visual mesh filename=/unitree/livox_mapping/robots/g1_description/meshes/torso_l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
- link waist_roll_link: geometry visual mesh filename=/unitree/livox_mapping/robots/g1_description/meshes/waist_r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
- link waist_yaw_link: geometry visual mesh filename=/unitree/livox_mapping/robots/g1_description/meshes/waist_y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
Joints:
- added joint base_to_pelvis: type fixed, parent base_link, child pelvis, origin xyz=0 0 0 rpy=0 0 0

Commit message: made the hardcoded ones dynamic

File: robots/g1_description/g1_29dof_lock_waist_with_hand_rev_1_0.urdf (robot description, URDF)
Before this commit: robot g1_29dof_lock_waist_with_hand_rev_1_0, 54 links, 53 joints
Links:
- link head_link: geometry collision mesh filename=package://livox_mapping/robots/g1_description/meshes/head_l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; visual mesh filename=package://livox_mapping/robots/g1_description/meshes/head_l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
- link left_ankle_pitch_link: geometry collision mesh filename=package://livox_mapping/robots/g1_description/meshes/left_a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; visual mesh filename=package://livox_mapping/robots/g1_description/meshes/left_a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
- link left_ankle_roll_link: geometry collision sphere radius=0.005; collision sphere radius=0.005
- link left_elbow_link: geometry collision mesh filename=package://livox_mapping/robots/g1_description/meshes/left_e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; visual mesh filename=package://livox_mapping/robots/g1_description/meshes/left_e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
- link left_hand_index_0_link: geometry collision mesh filename=package://livox_mapping/robots/g1_description/meshes/left_h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; visual mesh filename=package://livox_mapping/robots/g1_description/meshes/left_h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
- link left_hand_index_1_link: geometry collision mesh filename=package://livox_mapping/robots/g1_description/meshes/left_h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; visual mesh filename=package://livox_mapping/robots/g1_description/meshes/left_h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
- link left_hand_middle_0_link: geometry collision mesh filename=package://livox_mapping/robots/g1_description/meshes/left_h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; visual mesh filename=package://livox_mapping/robots/g1_description/meshes/left_h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
- link left_hand_middle_1_link: geometry collision mesh filename=package://livox_mapping/robots/g1_description/meshes/left_h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; visual mesh filename=package://livox_mapping/robots/g1_description/meshes/left_h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
- link left_hand_palm_link: geometry collision mesh filename=package://livox_mapping/robots/g1_description/meshes/left_h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; visual mesh filename=package://livox_mapping/robots/g1_description/meshes/left_h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
- link left_hand_thumb_0_link: geometry collision mesh filename=package://livox_mapping/robots/g1_description/meshes/left_h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; visual mesh filename=package://livox_mapping/robots/g1_description/meshes/left_h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
- link left_hand_thumb_1_link: geometry collision box size=0.02 0.03 0.02; visual mesh filename=package://livox_mapping/robots/g1_description/meshes/left_h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
- link left_hand_thumb_2_link: geometry collision mesh filename=package://livox_mapping/robots/g1_description/meshes/left_h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; visual mesh filename=package://livox_mapping/robots/g1_description/meshes/left_h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
- link left_hip_pitch_link: geometry collision mesh filename=package://livox_mapping/robots/g1_description/meshes/left_h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; visual mesh filename=package://livox_mapping/robots/g1_description/meshes/left_h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
- link left_hip_roll_link: geometry collision mesh filename=package://livox_mapping/robots/g1_description/meshes/left_h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; visual mesh filename=package://livox_mapping/robots/g1_description/meshes/left_h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
- link left_hip_yaw_link: geometry collision mesh filename=package://livox_mapping/robots/g1_description/meshes/left_h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; visual mesh filename=package://livox_mapping/robots/g1_description/meshes/left_h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
- link left_knee_link: geometry collision mesh filename=package://livox_mapping/robots/g1_description/meshes/left_k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; visual mesh filename=package://livox_mapping/robots/g1_description/meshes/left_k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
- link left_shoulder_pitch_link: geometry collision cylinder length=0.05 radius=0.03; visual mesh filename=package://livox_mapping/robots/g1_description/meshes/left_s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
- link left_shoulder_roll_link: geometry collision cylinder length=0.03 radius=0.03; visual mesh filename=package://livox_mapping/robots/g1_description/meshes/left_s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
- link left_shoulder_yaw_link: geometry collision mesh filename=package://livox_mapping/robots/g1_description/meshes/left_s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; visual mesh filename=package://livox_mapping/robots/g1_description/meshes/left_s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
- link left_wrist_pitch_link: geometry collision mesh filename=package://livox_mapping/robots/g1_description/meshes/left_w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; visual mesh filename=package://livox_mapping/robots/g1_description/meshes/left_w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
- link left_wrist_roll_link: geometry collision mesh filename=package://livox_mapping/robots/g1_description/meshes/left_w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; visual mesh filename=package://livox_mapping/robots/g1_description/meshes/left_w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
- link left_wrist_yaw_link: geometry collision mesh filename=package://livox_mapping/robots/g1_description/meshes/left_w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; visual mesh filename=package://livox_mapping/robots/g1_description/meshes/left_w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
- link logo_link: geometry collision mesh filename=package://livox_mapping/robots/g1_description/meshes/logo_l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; visual mesh filename=package://livox_mapping/robots/g1_description/meshes/logo_l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
- link pelvis: geometry visual mesh filename=package://livox_mapping/robots/g1_description/meshes/pelvis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
- link pelvis_contour_link: geometry collision mesh filename=package://livox_mapping/robots/g1_description/meshes/pelvis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; visual mesh filename=package://livox_mapping/robots/g1_description/meshes/pelvis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
- link right_ankle_pitch_link: geometry collision mesh filename=package://livox_mapping/robots/g1_description/meshes/right_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; visual mesh filename=package://livox_mapping/robots/g1_description/meshes/right_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
- link right_ankle_roll_link: geometry collision sphere radius=0.005; collision sphere radius=0.005
- link right_elbow_link: geometry collision mesh filename=package://livox_mapping/robots/g1_description/meshes/right_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; visual mesh filename=package://livox_mapping/robots/g1_description/meshes/right_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
- link right_hand_index_0_link: geometry collision mesh filename=package://livox_mapping/robots/g1_description/meshes/right_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; visual mesh filename=package://livox_mapping/robots/g1_description/meshes/right_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
- link right_hand_index_1_link: geometry collision mesh filename=package://livox_mapping/robots/g1_description/meshes/right_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; visual mesh filename=package://livox_mapping/robots/g1_description/meshes/right_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
- link right_hand_middle_0_link: geometry collision mesh filename=package://livox_mapping/robots/g1_description/meshes/right_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; visual mesh filename=package://livox_mapping/robots/g1_description/meshes/right_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
- link right_hand_middle_1_link: geometry collision mesh filename=package://livox_mapping/robots/g1_description/meshes/right_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; visual mesh filename=package://livox_mapping/robots/g1_description/meshes/right_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
- link right_hand_palm_link: geometry collision mesh filename=package://livox_mapping/robots/g1_description/meshes/right_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; visual mesh filename=package://livox_mapping/robots/g1_description/meshes/right_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
- link right_hand_thumb_0_link: geometry collision mesh filename=package://livox_mapping/robots/g1_description/meshes/right_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; visual mesh filename=package://livox_mapping/robots/g1_description/meshes/right_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
- link right_hand_thumb_1_link: geometry collision box size=0.02 0.03 0.02; visual mesh filename=package://livox_mapping/robots/g1_description/meshes/right_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
- link right_hand_thumb_2_link: geometry collision mesh filename=package://livox_mapping/robots/g1_description/meshes/right_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; visual mesh filename=package://livox_mapping/robots/g1_description/meshes/right_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
- link right_hip_pitch_link: geometry collision mesh filename=package://livox_mapping/robots/g1_description/meshes/right_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; visual mesh filename=package://livox_mapping/robots/g1_description/meshes/right_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
- link right_hip_roll_link: geometry collision mesh filename=package://livox_mapping/robots/g1_description/meshes/right_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; visual mesh filename=package://livox_mapping/robots/g1_description/meshes/right_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
- link right_hip_yaw_link: geometry collision mesh filename=package://livox_mapping/robots/g1_description/meshes/right_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; visual mesh filename=package://livox_mapping/robots/g1_description/meshes/right_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
- link right_knee_link: geometry collision mesh filename=package://livox_mapping/robots/g1_description/meshes/right_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; visual mesh filename=package://livox_mapping/robots/g1_description/meshes/right_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
- link right_shoulder_pitch_link: geometry collision cylinder length=0.05 radius=0.03; visual mesh filename=package://livox_mapping/robots/g1_description/meshes/right_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
- link right_shoulder_roll_link: geometry collision cylinder length=0.03 radius=0.03; visual mesh filename=package://livox_mapping/robots/g1_description/meshes/right_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
- link right_shoulder_yaw_link: geometry collision mesh filename=package://livox_mapping/robots/g1_description/meshes/right_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; visual mesh filename=package://livox_mapping/robots/g1_description/meshes/right_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
- link right_wrist_pitch_link: geometry collision mesh filename=package://livox_mapping/robots/g1_description/meshes/right_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; visual mesh filename=package://livox_mapping/robots/g1_description/meshes/right_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
- link right_wrist_roll_link: geometry collision mesh filename=package://livox_mapping/robots/g1_description/meshes/right_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; visual mesh filename=package://livox_mapping/robots/g1_description/meshes/right_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
- link right_wrist_yaw_link: geometry collision mesh filename=package://livox_mapping/robots/g1_description/meshes/right_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; visual mesh filename=package://livox_mapping/robots/g1_description/meshes/right_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
- link torso_link: geometry collision mesh filename=package://livox_mapping/robots/g1_description/meshes/torso_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; visual mesh filename=package://livox_mapping/robots/g1_description/meshes/torso_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
- link waist_roll_link: geometry visual mesh filename=package://livox_mapping/robots/g1_description/meshes/waist_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
- link waist_yaw_link: geometry visual mesh filename=package://livox_mapping/robots/g1_description/meshes/waist_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
